File: pga103_active_dipole/v1/rev-/pga103_active_dipole.sch (KiCad schematic (older format))
At the start: 31 parts, among them J1 RF OUT, U1 SPX3819M5-L-5-0, U2 PGA-103

Commit message: updated bias-t values
Parts:
- L1: value 27nH -> 470uH
- L2: value 27nH -> 56nH
Changed lines of the file:
@@
 P 8100 3250
 F 0 "L1" H 8153 3296 50  0000 L CNN
-F 1 "27nH" H 8153 3205 50  0000 L CNN
+F 1 "470uH" H 8153 3205 50  0000 L CNN
 F 2 "digikey-footprints:0805" H 8100 3250 50  0001 C CNN
 F 3 "~" H 8100 3250 50  0001 C CNN
@@
 P 6900 3650
 F 0 "L2" H 6953 3696 50  0000 L CNN
-F 1 "27nH" H 6953 3605 50  0000 L CNN
+F 1 "56nH" H 6953 3605 50  0000 L CNN
 F 2 "digikey-footprints:0805" H 6900 3650 50  0001 C CNN
 F 3 "~" H 6900 3650 50  0001 C CNN
